File: WarpSE-Overclocking-Board.kicad_pcb (KiCad board)
At the start: 4 copper layers, 33.5 x 23.6 mm, 26 parts, among them J1 DBG, SW1 CFG, U1 30M, U2 32M, U3 36M, U4 74LVC1G08GW, U5 74LVC1G08GW, U6 74LVC1G86GW, U7 74LVC1G02GW, U8 XC6206PxxxMR

Commit message: As sent to JLC
Parts:
- added G***: LOGO, LOGO, B.Cu at (83.1, 111.3)
- U2: value 32M -> 33M
- U8: value XC6206PxxxMR -> XC6206P332MR
- moved C1 0.10 mm to (104.9, 114.3)
Connections:
- net /EN32 renamed /EN33
- J1 pad 5: /DBG0_~{ROMWS} -> /DBG1_~{RAMWS}
- J1 pad 6: /DBG1_~{RAMWS} -> /DBG0_~{ROMWS}
Routing:
- net /DBG1_~{RAMWS}: track 16.5 -> 46.9 mm
- net /DBG0_~{ROMWS}: track 13.0 -> 37.8 mm
- net /DBG4_~{IOWS}: track 14.9 -> 30.0 mm
- net /CLKSEL0: track 18.2 -> 17.3 mm, vias 3 -> 0
- net /CLKSEL1: track 22.3 -> 21.4 mm
- net GND: vias 71 -> 76
- added copper zone on In2.Cu, net GND
Other:
- board text added: "WarpSE Overclocker"
- board text added: "for GW4410A"
