File: WarpSE-Overclocking-Board.kicad_sch (KiCad schematic)
At the start: 26 parts, among them J1 DBG, SW1 CFG, U1 30M, U2 32M, U3 36M, U4 74LVC1G08GW, U5 74LVC1G08GW, U6 74LVC1G86GW, U7 74LVC1G02GW, U8 XC6206PxxxMR

Commit message: As sent to JLC
Parts:
- U2: value 32M -> 33M
- U8: value XC6206PxxxMR -> XC6206P332MR
Connections:
- net DBG0_~{ROMWS}: now also J1.6 (Pin_6); no longer J1.5 (Pin_5)
- net DBG1_~{RAMWS}: now also J1.5 (Pin_5); no longer J1.6 (Pin_6)
- net EN32 renamed EN33
Other:
- title: WarpSE-OC (GW4411A) -> WarpSE-OC (GW4490A)
Changed lines of the file:
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@@
 	(generator "eeschema")
 	(generator_version "8.0")
-	(paper "A4")
+	(paper "USLetter")
 	(title_block
-		(title "WarpSE-OC (GW4411A)")
-		(date "2024-10-19")
+		(title "WarpSE-OC (GW4490A)")
+		(date "2025-01-05")
 		(rev "1.0")
 		(company "Garrett's Workshop")
@@
 		)
 	)
-	(label "EN32"
+	(label "EN33"
 		(at 176.53 83.82 0)
 		(fields_autoplaced yes)
@@
 	)
 	(label "DBG0_~{ROMWS}"
-		(at 106.68 170.18 0)
+		(at 93.98 170.18 180)
 		(fields_autoplaced yes)
 		(effects
@@
 				(size 1.27 1.27)
 			)
-			(justify left bottom)
+			(justify right bottom)
 		)
 	)
@@
 	)
 	(label "DBG1_~{RAMWS}"
-		(at 93.98 170.18 180)
+		(at 106.68 170.18 0)
 		(fields_autoplaced yes)
 		(effects
@@
 				(size 1.27 1.27)
 			)
-			(justify right bottom)
+			(justify left bottom)
 		)
 	)
@@
 			)
 		)
-		(property "Value" "XC6206PxxxMR"
+		(property "Value" "XC6206P332MR"
 			(at 41.91 104.14 0)
 			(effects
@@
 			)
 		)
-		(property "Value" "32M"
+		(property "Value" "33M"
 			(at 193.04 90.17 0)
 			(effects
